File: Schematic/YM2151_STM32_VGM.sch (KiCad schematic (older format))
At the start: 52 parts, among them J1 DM3CS-SF (Micro SD Card Slot), J2 Jack_DC+12V, J3 JACK_TRS_6PINS, J4 USB_B, SW1 PWR_SWITCH, SW2 MUTE_SWITCH, SW3 PREV, SW4 RAND, SW5 NEXT, SW6 LOOP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

Commit message: Corrected SD card on schematic and board. Added button control
Parts:
- removed J1: DM3CS-SF (Micro SD Card Slot), Connector_Card:SD_TE_2041021, symbol DM3CS-SF
- added J1: SD_Card, Connector_Card:SD_TE_2041021, symbol SD_Card
Connections:
- wire segments 171 -> 170
